File: hardware/reflectance_array.kicad_pcb (KiCad board)
At the start: 2 copper layers, 64 x 20 mm, 19 parts, among them U1 AP3019A, U2 ITR1502SR40A, U3 ITR1502SR40A, U4 ITR1502SR40A, U5 ITR1502SR40A, U6 ITR1502SR40A, U7 ITR1502SR40A, U8 ATtiny1616-M

Commit message: first draft version
Parts:
- added G***: LOGO, shurik-personal:my_logo, B.Cu at (118.5, 91.0)
- added J1: Conn_01x04_Pin, Connector_JST:JST_SH_SM04B-SRSS-TB_1x04-1MP_P1.00mm_Horizontal, B.Cu at (130.0, 90.0)
- added J2: Conn_01x04_Pin, shurik-personal:connector-4p-generic-nosilk, B.Cu at (126.2, 97.5)
- added JP1: SolderJumper_2_Open, Jumper:SolderJumper-2_P1.3mm_Open_TrianglePad1.0x1.5mm, B.Cu at (143.2, 91.5)
- added JP2: SolderJumper_2_Open, Jumper:SolderJumper-2_P1.3mm_Open_TrianglePad1.0x1.5mm, B.Cu at (143.2, 88.8)
- added R8: 3.3K, Resistor_SMD:R_0603_1608Metric, F.Cu at (144.5, 94.0)
- added R9: 3.3K, Resistor_SMD:R_0603_1608Metric, F.Cu at (146.5, 94.0)
- added REF**: MountingHole_3.2mm_M3, MountingHole:MountingHole_3.2mm_M3, F.Cu at (110.0, 90.0)
- added REF**: MountingHole_3.2mm_M3, MountingHole:MountingHole_3.2mm_M3, F.Cu at (150.0, 90.0)
- added TP1: TestPoint, TestPoint:TestPoint_Pad_D1.5mm, B.Cu at (145.2, 97.8)
- added TP2: TestPoint, TestPoint:TestPoint_Pad_D1.5mm, B.Cu at (140.2, 97.8)
- added TP3: TestPoint, TestPoint:TestPoint_Pad_D1.5mm, B.Cu at (142.7, 97.8)
- added kibuzzard-67E071FA: G***, kibuzzard-67E071FA, F.Cu at (115.0, 80.8)
- added kibuzzard-67E07232: G***, kibuzzard-67E07232, F.Cu at (125.0, 80.8)
- added kibuzzard-67E07257: G***, kibuzzard-67E07257, F.Cu at (105.0, 80.8)
- added kibuzzard-67E072A1: G***, kibuzzard-67E072A1, F.Cu at (135.0, 80.8)
- added kibuzzard-67E072AD: G***, kibuzzard-67E072AD, F.Cu at (145.0, 80.8)
- added kibuzzard-67E072BD: G***, kibuzzard-67E072BD, F.Cu at (155.0, 80.8)
- added kibuzzard-67E0733D: G***, kibuzzard-67E0733D, B.Cu at (115.0, 81.0)
- added kibuzzard-67E0734D: G***, kibuzzard-67E0734D, B.Cu at (105.0, 81.0)
- added kibuzzard-67E0737D: G***, kibuzzard-67E0737D, B.Cu at (125.0, 81.0)
- added kibuzzard-67E07391: G***, kibuzzard-67E07391, B.Cu at (145.0, 81.0)
- added kibuzzard-67E073A3: G***, kibuzzard-67E073A3, B.Cu at (135.0, 81.0)
- added kibuzzard-67E073B0: G***, kibuzzard-67E073B0, B.Cu at (155.0, 81.0)
- L1: footprint Inductor_SMD:L_Taiyo-Yuden_NR-40xx -> Inductor_SMD:L_Sunlord_SWPA5020S
- R2, R3, R4, R5, R6, R7: value 10K -> 1.5K
- moved C2 69.4 mm to (115.8, 94.8), turned to -90 degrees
- moved C1 62.6 mm to (124.0, 94.0), turned to 90 degrees
- moved R1 60.6 mm to (122.6, 90.4), turned to -90 degrees
- moved C3 17.5 mm to (142.5, 94.0), turned to -90 degrees
- moved U1 15.2 mm to (119.5, 90.5), turned to 180 degrees
- moved U8 9.47 mm to (138.5, 94.0), turned to 180 degrees
- moved L1 4.74 mm to (119.5, 95.5)
Connections:
- C1 pad 1: VCC -> +3V3
- L1 pad 1: VCC -> +3V3
- R2 pad 2: Net-(R2-Pad2) -> /A1
- R3 pad 2: Net-(R3-Pad2) -> /A2
- R4 pad 2: Net-(R4-Pad2) -> /A3
- R5 pad 2: Net-(R5-Pad2) -> /A4
- R6 pad 2: Net-(R6-Pad2) -> /A5
- R7 pad 2: Net-(R7-Pad2) -> /A6
- U1 pad 6: VCC -> +3V3
- U2 pad 2: Net-(R2-Pad2) -> /A1
- U3 pad 2: Net-(R3-Pad2) -> /A2
- U4 pad 2: Net-(R4-Pad2) -> /A3
- U5 pad 2: Net-(R5-Pad2) -> /A4
- U6 pad 2: Net-(R6-Pad2) -> /A5
- U7 pad 2: Net-(R7-Pad2) -> /A6
- U8 pad 10: unconnected-(U8-PB4-Pad10) -> /A1
- U8 pad 11: unconnected-(U8-PB3-Pad11) -> /LED_ENABLE
- U8 pad 13: unconnected-(U8-PB1-Pad13) -> /SDA
- U8 pad 14: unconnected-(U8-PB0-Pad14) -> /SCL
- U8 pad 19: unconnected-(U8-~{RESET}/PA0-Pad19) -> /UPDI
- U8 pad 5: unconnected-(U8-PA4-Pad5) -> /A6
- U8 pad 6: unconnected-(U8-PA5-Pad6) -> /A5
- U8 pad 7: unconnected-(U8-PA6-Pad7) -> /A4
- U8 pad 8: unconnected-(U8-PA7-Pad8) -> /A3
- U8 pad 9: unconnected-(U8-PB5-Pad9) -> /A2
Routing:
- net +3V3: track 0.00 -> 122.9 mm, vias 0 -> 7
- net /FB: track 0.00 -> 55.7 mm
- net /A1: track 0.00 -> 38.3 mm
- net /SDA: track 0.00 -> 31.6 mm, vias 0 -> 1
- net /VCC_LED: track 0.00 -> 30.2 mm
- net /A2: track 0.00 -> 28.9 mm
- net /SCL: track 0.00 -> 24.5 mm, vias 0 -> 1
- net /A6: track 0.00 -> 22.1 mm
- net /LED_ENABLE: track 0.00 -> 21.4 mm
- net GNDREF: track 0.00 -> 19.0 mm, vias 0 -> 9
- net /A3: track 0.00 -> 16.6 mm
- net /A5: track 0.00 -> 12.8 mm
- net /A4: track 0.00 -> 9.40 mm
- net Net-(U6-K): track 0.00 -> 7.60 mm
- net Net-(U5-K): track 0.00 -> 7.60 mm
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Other:
- outline, holes or cut-outs redrawn
- board text added: "3V3"
- board text added: "GND"
- board text added: "I2C pullups"
- board text added: "SCL"
- board text added: "SDA"
- board text added: "UPDI"

Commit message: version 0.1
Parts:
- removed kibuzzard-67E071FA: G***, kibuzzard-67E071FA
- removed kibuzzard-67E07232: G***, kibuzzard-67E07232
- removed kibuzzard-67E07257: G***, kibuzzard-67E07257
- removed kibuzzard-67E072A1: G***, kibuzzard-67E072A1
- removed kibuzzard-67E072AD: G***, kibuzzard-67E072AD
- removed kibuzzard-67E072BD: G***, kibuzzard-67E072BD
- removed kibuzzard-67E0733D: G***, kibuzzard-67E0733D
- removed kibuzzard-67E0734D: G***, kibuzzard-67E0734D
- removed kibuzzard-67E0737D: G***, kibuzzard-67E0737D
- removed kibuzzard-67E07391: G***, kibuzzard-67E07391
- removed kibuzzard-67E073A3: G***, kibuzzard-67E073A3
- removed kibuzzard-67E073B0: G***, kibuzzard-67E073B0
- added J3: Conn_01x01_Pin, shurik-personal:connector-1p-generic-nosilk, F.Cu at (103.8, 87.8)
- added J4: Conn_01x01_Pin, shurik-personal:connector-1p-generic-nosilk, F.Cu at (120.0, 83.8)
- added J5: Conn_01x01_Pin, shurik-personal:connector-1p-generic-nosilk, F.Cu at (130.0, 83.8)
- added J6: Conn_01x01_Pin, shurik-personal:connector-1p-generic-nosilk, F.Cu at (156.8, 88.0)
- added kibuzzard-67E182C9: G***, kibuzzard-67E182C9, B.Cu at (105.0, 81.0)
- added kibuzzard-67E182D6: G***, kibuzzard-67E182D6, B.Cu at (115.0, 81.0)
- added kibuzzard-67E182E1: G***, kibuzzard-67E182E1, B.Cu at (125.0, 81.0)
- added kibuzzard-67E182EE: G***, kibuzzard-67E182EE, B.Cu at (135.0, 81.0)
- added kibuzzard-67E182F6: G***, kibuzzard-67E182F6, B.Cu at (145.0, 81.0)
- added kibuzzard-67E1830C: G***, kibuzzard-67E1830C, B.Cu at (155.0, 81.0)
- added kibuzzard-67E1831D: G***, kibuzzard-67E1831D, F.Cu at (105.0, 80.8)
- added kibuzzard-67E18323: G***, kibuzzard-67E18323, F.Cu at (115.0, 80.8)
- added kibuzzard-67E18328: G***, kibuzzard-67E18328, F.Cu at (125.0, 80.8)
- added kibuzzard-67E1832E: G***, kibuzzard-67E1832E, F.Cu at (135.0, 80.8)
- added kibuzzard-67E18337: G***, kibuzzard-67E18337, F.Cu at (145.0, 80.8)
- added kibuzzard-67E18343: G***, kibuzzard-67E18343, F.Cu at (155.0, 80.8)
- J1: moved to F.Cu
- R1: value 10 -> 12
- R7: value 1.5K -> 10K
- moved J2 7.50 mm to (126.2, 90.0)
- moved R2 7.00 mm to (102.0, 85.0), turned to 90 degrees
- moved R3 7.00 mm to (112.0, 85.0), turned to 90 degrees
- moved R4 7.00 mm to (122.0, 85.0), turned to 90 degrees
- moved R5 7.00 mm to (132.0, 85.0), turned to 90 degrees
- moved R6 7.00 mm to (142.0, 85.0), turned to 90 degrees
- moved J1 4.25 mm to (130.0, 94.2)
Connections:
- R2 pad 1: +3V3 -> /A1
- R2 pad 2: /A1 -> GNDREF
- R3 pad 1: +3V3 -> /A2
- R3 pad 2: /A2 -> GNDREF
- R4 pad 1: +3V3 -> /A3
- R4 pad 2: /A3 -> GNDREF
- R5 pad 1: +3V3 -> /A4
- R5 pad 2: /A4 -> GNDREF
- R6 pad 1: +3V3 -> /A5
- R6 pad 2: /A5 -> GNDREF
- U2 pad 1: GNDREF -> /A1
- U2 pad 2: /A1 -> +3V3
- U3 pad 1: GNDREF -> /A2
- U3 pad 2: /A2 -> +3V3
- U4 pad 1: GNDREF -> /A3
- U4 pad 2: /A3 -> +3V3
- U5 pad 1: GNDREF -> /A4
- U5 pad 2: /A4 -> +3V3
- U6 pad 1: GNDREF -> /A5
- U6 pad 2: /A5 -> +3V3
Routing:
- net +3V3: track 122.9 -> 108.8 mm, vias 7 -> 8
- net /A3: track 16.6 -> 24.8 mm
- net /A4: track 9.40 -> 15.2 mm
- net /SCL: track 24.5 -> 21.6 mm
- net /A6: track 22.1 -> 24.7 mm
- net /A1: track 38.3 -> 40.5 mm
- net /A5: track 12.8 -> 10.9 mm
- net /SDA: track 31.6 -> 29.9 mm, vias 1 -> 0
- net /A2: track 28.9 -> 30.2 mm
- net /LED_ENABLE: track 21.4 -> 22.7 mm
- net /FB: track 55.7 -> 56.8 mm
- net /VCC_LED: track 30.2 -> 31.0 mm
- net GNDREF: track 19.0 -> 19.8 mm
Other:
- outline, holes or cut-outs redrawn

Commit message: version 1.0
Parts:
- removed the J3 at (103.8, 87.8)
- removed J4, J5: Conn_01x01_Pin, shurik-personal:connector-1p-generic-nosilk
- JP2: value SolderJumper_2_Open -> SolderJumper_3_Bridged123; footprint Jumper:SolderJumper-2_P1.3mm_Open_TrianglePad1.0x1.5mm -> shurik-personal:SolderJumper-3_P1.3mm_Bridged123_RoundedPad1.0x1.5mm
- R2, R3, R4, R5, R6: value 1.5K -> 10K
- TP1: renamed from TP2; moved to F.Cu
- TP2: renamed from TP3; moved to F.Cu
- TP3: renamed from TP1; moved to F.Cu
- moved J1 52.3 mm to (104.5, 88.2)
- moved TP1 19.0 mm to (157.5, 90.0), turned to 0 degrees
- moved TP2 15.7 mm to (157.5, 92.5), turned to 0 degrees
- moved TP3 12.6 mm to (157.5, 95.0), turned to 0 degrees
- moved JP1 8.36 mm to (149.8, 96.8)
- moved R8 7.04 mm to (152.0, 84.2)
- moved R2 6.05 mm to (108.0, 84.2), turned to -90 degrees
- moved R3 6.05 mm to (118.0, 84.2), turned to -90 degrees
- moved R4 6.05 mm to (128.0, 84.2), turned to -90 degrees
- moved R5 6.05 mm to (138.0, 84.2), turned to -90 degrees
- moved R6 6.05 mm to (148.0, 84.2), turned to -90 degrees
- moved G*** 2.06 mm to (118.0, 93.0), turned to 180 degrees
- moved JP2 1.51 mm to (144.2, 89.9), turned to 90 degrees
- moved J3 1.00 mm to (126.2, 89.0)
- moved kibuzzard-67E1831D 0.25 mm to (105.0, 81.0)
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- renumbered J6 to J1, J1 to J2, J2 to J3, R8 to R7, R7 to R8, U8 to U4, U4 to U5, U5 to U6, U6 to U7, U7 to U8
Connections:
- J1 pad 1: /A6 -> /S0
- JP1 pad 1: Net-(JP1-A) -> GNDREF
- JP1 pad 2: +3V3 -> /I2C_ADDR
- JP2 pad 1: Net-(JP2-A) -> +3V3
- R2 pad 1: /A1 -> +3V3
- R2 pad 2: GNDREF -> /S0
- R3 pad 1: /A2 -> +3V3
- R3 pad 2: GNDREF -> /S1
- R4 pad 1: /A3 -> +3V3
- R4 pad 2: GNDREF -> /S2
- R5 pad 1: /A4 -> +3V3
- R5 pad 2: GNDREF -> /S3
- R6 pad 1: /A5 -> +3V3
- R6 pad 2: GNDREF -> /S4
- R7 pad 1: Net-(JP1-A) -> +3V3
- R8 pad 2: /A6 -> /S5
- R9 pad 1: Net-(JP2-A) -> +3V3
- U2 pad 1: /A1 -> GNDREF
- U2 pad 2: +3V3 -> /S0
- U3 pad 1: /A2 -> GNDREF
- U3 pad 2: +3V3 -> /S1
- U4 pad 10: /A1 -> /S0
- U4 pad 17: unconnected-(U8-PC2-Pad17) -> /I2C_ADDR
- U4 pad 5: /A6 -> /S5
- U4 pad 6: /A5 -> /S4
- U4 pad 7: /A4 -> /S3
- U4 pad 8: /A3 -> /S2
- U4 pad 9: /A2 -> /S1
- U5 pad 1: /A3 -> GNDREF
- U5 pad 2: +3V3 -> /S2
- U6 pad 1: /A4 -> GNDREF
- U6 pad 2: +3V3 -> /S3
- U7 pad 1: /A5 -> GNDREF
- U7 pad 2: +3V3 -> /S4
- U8 pad 2: /A6 -> /S5
Routing:
- net /S0: track 0.00 -> 41.1 mm
- net /A1: track 40.5 -> 0.00 mm
- net /A2: track 30.2 -> 0.00 mm
- net /S1: track 0.00 -> 28.9 mm
- net /A3: track 24.8 -> 0.00 mm
- net /A6: track 24.7 -> 0.00 mm
- net /S5: track 0.00 -> 22.3 mm
- net /UPDI: track 2.86 -> 22.4 mm, vias 1 -> 2
- net /S2: track 0.00 -> 17.5 mm
- net +3V3: track 108.8 -> 126.1 mm, vias 8 -> 10
- net /A4: track 15.2 -> 0.00 mm
- net /I2C_ADDR: track 0.00 -> 12.6 mm, vias 0 -> 1
- net /S4: track 0.00 -> 12.2 mm
- net /A5: track 10.9 -> 0.00 mm
- net /S3: track 0.00 -> 10.0 mm
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Other:
- board size 64 x 20 mm -> 60 x 20 mm
- board text added: "I2C addr"
- board text added: "Line array v1.0"
- board text added: "github.com/shurik179"
