File: hardware/reflectance_array.kicad_sch (KiCad schematic)
At the start: 19 parts, among them U10 AP3019A, U2 ITR1502SR40A, U3 ITR1502SR40A, U4 ITR1502SR40A, U5 ITR1502SR40A, U6 ITR1502SR40A, U7 ITR1502SR40A, U8 ATtiny1616-M

Commit message: first draft version
Parts:
- added J1: Conn_01x04_Pin, Connector_JST:JST_SH_SM04B-SRSS-TB_1x04-1MP_P1.00mm_Horizontal, symbol Connector:Conn_01x04_Pin
- added J2: Conn_01x04_Pin, shurik-personal:connector-4p-generic-nosilk, symbol Connector:Conn_01x04_Pin
- added JP1, JP2: SolderJumper_2_Open, Jumper:SolderJumper-2_P1.3mm_Open_TrianglePad1.0x1.5mm, symbol Jumper:SolderJumper_2_Open
- added R8, R9: 3.3K, Resistor_SMD:R_0603_1608Metric, symbol Device:R_Small
- added TP1, TP2, TP3: TestPoint, TestPoint:TestPoint_Pad_D1.5mm, symbol Connector:TestPoint
- L1: footprint Inductor_SMD:L_Taiyo-Yuden_NR-40xx -> Inductor_SMD:L_Sunlord_SWPA5020S; LCSC C2880384 -> C96915
- R1, R2, R4, R5, R6, R7: value 10K -> 1.5K; LCSC C25804 -> C22843
- R15: LCSC C319921 -> C22859
Connections:
- net VCC is gone; now on net +3V3: C8.1, L1.1, U10.6 (VIN)
- net +3V3: now also J1.2 (Pin_2), J2.2 (Pin_2), JP1.2 (B), JP2.2 (B), TP3.1
- net GNDREF: now also J1.1 (Pin_1), J2.1 (Pin_1), TP1.1
- net LED_ENABLE: now also U8.11 (PB3)
- net A5: now reaches R6.2, U6.2
- net A5: now also U8.6 (PA5)
- net A6: now reaches R7.2, U7.2
- net A6: now also U8.5 (PA4)
- net A1: now reaches R1.2, U2.2
- net A1: now also U8.10 (PB4)
- net A4: now reaches R5.2, U5.2
- net A4: now also U8.7 (PA6)
- net A3: now reaches R4.2, U4.2
- net A3: now also U8.8 (PA7)
- net SDA: now reaches U8.13 (PB1)
- net SDA: now also J1.3 (Pin_3), J2.3 (Pin_3), R9.2
- net SCL: now reaches U8.14 (PB0)
- net SCL: now also J1.4 (Pin_4), J2.4 (Pin_4), R8.2
- net UPDI: now reaches U8.19 (~{RESET}/PA0)
- net UPDI: now also TP2.1
- net A2: now reaches U8.9 (PB5)
- net A2: now also R2.2, U3.2
- new net: JP2.1 (A), R9.1
- new net: JP1.1 (A), R8.1

Commit message: version 0.1
Parts:
- added J3, J4, J5, J6: Conn_01x01_Pin, shurik-personal:connector-1p-generic-nosilk, symbol Connector:Conn_01x01_Pin
- J1: LCSC (none) -> C160404
- R15: value 10 -> 12; LCSC C22859 -> C245909
- R7: value 1.5K -> 10K; LCSC C22843 -> C25804
Connections:
- net +3V3: now also U2.2, U3.2, U4.2, U5.2, U6.2; no longer R1.1, R2.1, R4.1, R5.1, R6.1
- net A1: now also R1.1, U2.1, J3.1 (Pin_1); no longer R1.2, U2.2
- net A2: now also R2.1, U3.1; no longer R2.2, U3.2
- net A3: now also R4.1, U4.1, J4.1 (Pin_1); no longer R4.2, U4.2
- net A4: now also R5.1, U5.1, J5.1 (Pin_1); no longer R5.2, U5.2
- net A5: now also R6.1, U6.1; no longer R6.2, U6.2
- net A6: now also J6.1 (Pin_1)
- net GNDREF: now also R1.2, R2.2, R4.2, R5.2, R6.2; no longer U2.1, U3.1, U4.1, U5.1, U6.1
Other:
- moved on the sheet: R1, R2, R4, R5, R6

Commit message: version 1.0
Parts:
- removed J3, J4, J5: Conn_01x01_Pin, shurik-personal:connector-1p-generic-nosilk, symbol Connector:Conn_01x01_Pin
- removed JP2: SolderJumper_2_Open, Jumper:SolderJumper-2_P1.3mm_Open_TrianglePad1.0x1.5mm, symbol Jumper:SolderJumper_2_Open
- removed R1: 1.5K, Resistor_SMD:R_0603_1608Metric, symbol Device:R_Small
- added JP2: SolderJumper_3_Bridged123, shurik-personal:SolderJumper-3_P1.3mm_Bridged123_RoundedPad1.0x1.5mm, symbol Jumper:SolderJumper_3_Bridged123
- added R3: 10K, Resistor_SMD:R_0603_1608Metric, symbol Device:R_Small
- R2, R4, R5, R6: value 1.5K -> 10K; LCSC C22843 -> C25804
- renumbered J6 to J1, J1 to J2, J2 to J3, R8 to R7, R7 to R8, TP2 to TP1, TP3 to TP2, TP1 to TP3, U8 to U4, U4 to U5, U5 to U6, U6 to U7, U7 to U8
Connections:
- net +3V3: now also R2.1, R4.1, R5.1, R6.1, R7.1, R9.1, JP2.1 (A), JP2.2 (C), JP2.3 (B), R3.1; no longer JP1.2 (B), U2.2, U3.2, U5.2, U6.2, U7.2
- net GNDREF: now also JP1.1 (A), U2.1, U3.1, U5.1, U6.1, U7.1; no longer R2.2, R4.2, R5.2, R6.2
- net I2C_ADDR: now reaches U4.17 (PC2)
- net I2C_ADDR: now also JP1.2 (B)
- net A1 renamed S0
- net S0: now also J1.1 (Pin_1), R2.2, U2.2; no longer U2.1
- removed net A2: R2.1, U3.1, U4.9 (PB5)
- removed net A3: R4.1, U4.8 (PA7), U5.1
- removed net A4: R5.1, U4.7 (PA6), U6.1
- removed net A5: R6.1, U4.6 (PA5), U7.1
- net A6 renamed S5
- net S5: no longer J1.1 (Pin_1)
- new net S1: R3.2, U3.2, U4.9 (PB5)
- new net S2: R4.2, U4.8 (PA7), U5.2
- new net S3: R5.2, U4.7 (PA6), U6.2
- new net S4: R6.2, U4.6 (PA5), U7.2
Other:
- moved on the sheet: J1, U10
